Commit message: added and updated mapping

File: catkin_ws/src/my_robot/urdf/my_robot.xacro (robot description, xacro)
@@ -158,9 +158,28 @@
     </joint>
     <joint name="camera_optical_joint" type="fixed">
-      <origin xyz="0 0 0" rpy="-1.5707 0 -1.5707"/>
+      <origin xyz="0.23 0 0.05" rpy="0 0 0"/>
       <parent link="camera"/>
       <child link="camera_link_optical"/>
     </joint>
     <link name="camera_link_optical">
+      <collision>
+        <geometry>
+          <box size="0.05 0.02 0.02"/>
+        </geometry>
+        <origin xyz="0.03 0 -0.05" rpy="0 0 0"/>
+      </collision>
+      <inertial>
+        <mass value="0.1"/>
+        <inertia ixx="1e-6" ixy="0" ixz="0" iyy="1e-6" iyz="0" izz="1e-6"/>
+      </inertial>
+      <visual name="camera_visual">
+        <geometry>
+          <box size="0.05 0.02 0.02"/>
+        </geometry>
+        <origin xyz="0.03 0 -0.05" rpy="0 0 0"/>
+        <material name="CameraMaterial">
+          <color rgba="1.0 0.0 0.0 1.0"/>
+        </material>
+      </visual>
     </link>
     <gazebo reference="camera">

Commit message: updated mapping and added localization

File: catkin_ws/src/my_robot/urdf/my_robot.xacro (robot description, xacro)
@@ -163,23 +163,4 @@
     </joint>
     <link name="camera_link_optical">
-      <collision>
-        <geometry>
-          <box size="0.05 0.02 0.02"/>
-        </geometry>
-        <origin xyz="0.03 0 -0.05" rpy="0 0 0"/>
-      </collision>
-      <inertial>
-        <mass value="0.1"/>
-        <inertia ixx="1e-6" ixy="0" ixz="0" iyy="1e-6" iyz="0" izz="1e-6"/>
-      </inertial>
-      <visual name="camera_visual">
-        <geometry>
-          <box size="0.05 0.02 0.02"/>
-        </geometry>
-        <origin xyz="0.03 0 -0.05" rpy="0 0 0"/>
-        <material name="CameraMaterial">
-          <color rgba="1.0 0.0 0.0 1.0"/>
-        </material>
-      </visual>
     </link>
     <gazebo reference="camera">

Commit message: updated world and mapping

File: catkin_ws/src/my_robot/urdf/my_robot.xacro (robot description, xacro)
@@ -158,5 +158,5 @@
     </joint>
     <joint name="camera_optical_joint" type="fixed">
-      <origin xyz="0.23 0 0.05" rpy="0 0 0"/>
+      <origin xyz="0.23 0 0.05" rpy="-1.5707 0 -1.5707"/>
       <parent link="camera"/>
       <child link="camera_link_optical"/>
